File: pcb/nomad.kicad_pcb (KiCad board)
At the start: 2 copper layers, 65 x 120 mm, 78 parts, among them J1 USB_C_Receptacle_USB2.0_16P, J2 Conn_01x08_Pin, J3 Conn_Coaxial, J4 Conn_Coaxial, J5 Conn_01x02_Pin, Q2 2N7002, SW1 UP, SW2 DOWN, SW3 RIGHT, SW4 LEFT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

Commit message: Updating documentation
Parts:
- moved G*** 0.59 mm to (153.3, 139.8)
- moved G*** 0.18 mm to (126.9, 159.9)
Routing:
- net GND: vias 146 -> 158

Commit message: Finishing PCB
Parts:
- removed the REF** at (160.0, 50.1)
- removed the REF** at (105.0, 160.1)
- removed the REF** at (160.0, 160.2)
- removed the REF** at (105.0, 50.1)
- added REF**: MountingHole_2.2mm_M2_Pad, MountingHole:MountingHole_2.2mm_M2_Pad, F.Cu at (160.0, 50.0)
- added REF**: MountingHole_2.2mm_M2_Pad, MountingHole:MountingHole_2.2mm_M2_Pad, F.Cu at (105.0, 50.0)
- added REF**: MountingHole_2.2mm_M2_Pad, MountingHole:MountingHole_2.2mm_M2_Pad, F.Cu at (105.0, 160.1)
- added REF**: MountingHole_2.2mm_M2_Pad, MountingHole:MountingHole_2.2mm_M2_Pad, F.Cu at (160.0, 160.0)

Commit message: Fixing reversed polarity battery connector
Connections:
- J5 pad 1: +BATT -> GND
- J5 pad 2: GND -> +BATT
Routing:
- net +BATT: track 34.7 -> 35.7 mm
- net GND: track 25.4 -> 25.7 mm, vias 158 -> 183
Other:
- board text added: "+"
- board text added: "-"
- board text removed: "GPS"
- board text removed: "Lora Module"
